File: Hardware/OrionCore-H743XI/PowerModule.kicad_sch (KiCad schematic)
At the start: 0 parts

Commit message: feat: update dual qspi
Other:
- company: (none) -> Peakors
- title: (none) -> OrionCore
Changed lines of the file:
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@@
 	(generator_version "10.0")
 	(paper "A4")
+	(title_block
+		(title "OrionCore")
+		(date "2026-05-15")
+		(rev "V1.0")
+		(company "Peakors")
+	)
 )
